File: ESC_BOARD.brd (EAGLE design)
At the start: 139.2 x 39.9 mm, 34 parts, among them J1 TE_2351886-3-(VERT), J2 TE_2351886-3-(VERT), J3 TE_2351886-3-(VERT), J4 TE_2351886-3-(VERT), Y1 ECS-80-S-4X

Commit message: added pins for programing ESCs
Parts:
- removed JP1, JP2, JP3, JP4: JUMPER-SMT_2_NC_PASTE_SILK, SparkFun-Jumpers:SMT-JUMPER_2_NC_PASTE_SILK
- added J5, J6, J7, J8: (no value), SparkFun-Connectors:1X02
- moved U$5 4.68 mm to (59.4, 18.3), turned to 180 degrees
- moved C7 1.88 mm to (76.6, 31.1), turned to 270 degrees
- moved C10 0.13 mm to (72.3, 24.8)
Connections:
- net ESC_PWM_1: now also J5.1; no longer JP1.1
- net ESC_PWM_2: now also J6.1; no longer JP2.1
- net ESC_PWM_3: now also J7.1; no longer JP3.1
- net ESC_PWM_4: now also J8.1; no longer JP4.1
- net TIM3_CH1: now also J5.2; no longer JP1.2
- net TIM3_CH2: now also J6.2; no longer JP2.2
- net TIM3_CH3: now also J7.2; no longer JP3.2
- net TIM3_CH4: now also J8.2; no longer JP4.2
Routing:
- net ESC_PWM_1: track 20.7 -> 16.8 mm, vias 1 -> 0
- net TIM3_CH1: track 18.8 -> 15.8 mm
- net ESC_PWM_3: track 15.4 -> 12.8 mm, vias 1 -> 0
- net TIM3_CH4: track 8.62 -> 7.27 mm, vias 1 -> 0
- net ESC_PWM_2: track 12.7 -> 13.7 mm, vias 1 -> 0
- net !RST: track 55.1 -> 54.4 mm
- net RES_ID: track 25.8 -> 25.2 mm
- net ESC_PWM_4: track 16.1 -> 16.6 mm, vias 1 -> 0
- net TIM3_CH3: track 14.6 -> 14.1 mm, vias 1 -> 0
- net +12V: track 71.8 -> 71.6 mm, vias 34 -> 33
- net GND: vias 36 -> 40
